File: MetalDetector/KiCad/MetalDetector-Mirko-Mike.kicad_pcb (KiCad board)
At the start: 2 copper layers, 67.2 x 50 mm, 26 parts, among them J1 Conn_01x03_Pin, J2 Conn_01x03_Pin, J3 Display, Q1 2N2219, SW1 CAL, U2 MCP6281P or MCP6283P or TL081

Commit message: final PCB version 1, change earphone component on schematic
Parts:
- removed MountingHole3: MountingHole_4.3mm_M4, MountingHole:MountingHole_4.3mm_M4
- moved LS1 2.60 mm to (132.3, 107.0)
Connections:
- Q1 pad 3: Net-(LS1--) -> Net-(Q1-C)
Routing:
- net Net-(Q1-C): track 0.00 -> 32.4 mm
- net Net-(A1-+5V): track 74.2 -> 89.6 mm
- net Net-(J1-Pin_2): track 27.0 -> 19.3 mm, vias 1 -> 0
- net Net-(J2-Pin_1): track 63.4 -> 58.3 mm
- net GND: track 199.9 -> 201.2 mm
