File: MetalDetector/KiCad/MetalDetector-Mirko-Mike.kicad_sch (KiCad schematic)
At the start: 27 parts, among them J1 Conn_01x03_Pin, J1plug1 Conn_01x03_Socket, J2 Conn_01x03_Pin, J2plug1 Conn_01x03_Socket, J3 Display, Q1 2N2219, SW1 CAL, U2 MCP6281P or MCP6283P or TL081

Commit message: final PCB version 1, change earphone component on schematic
Parts:
- removed LS1: Earphone, SJ1_2503A:CONN_SJ1-2503A, symbol Device:Earphone
- added LS1: Earphone, SJ1_2503A:CONN_SJ1-2503A, symbol Connector_Audio:AudioJack2
Connections:
- net at A1.27 (+5V), J3.2 (Pin_2), U2.7 (V+): now also LS1.S
- net at Q1.3 (C): now also LS1.T
Changed lines of the file:
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@@
 	)
 	(junction
-		(at 49.53 125.73)
+		(at 115.57 46.99)
 		(diameter 0)
 		(color 0 0 0 0)
 	)
 	(junction
-		(at 215.9 97.79)
+		(at 49.53 125.73)
 		(diameter 0)
 		(color 0 0 0 0)
 	)
 	(junction
-		(at 74.93 124.46)
+		(at 215.9 97.79)
 		(diameter 0)
 		(color 0 0 0 0)
 	)
 	(junction
-		(at 115.57 46.99)
+		(at 74.93 124.46)
 		(diameter 0)
 		(color 0 0 0 0)
@@
 	(wire
 		(pts
+			(xy 115.57 46.99) (xy 220.98 46.99)
+		)
+		(stroke
+			(width 0)
+			(type default)
+		)
+	)
+	(wire
+		(pts
 			(xy 120.65 109.22) (xy 120.65 113.03)
 		)
@@
 	(wire
 		(pts
-			(xy 115.57 46.99) (xy 220.98 46.99)
+			(xy 234.95 137.16) (xy 245.11 137.16)
 		)
 		(stroke
@@
 	(wire
 		(pts
-			(xy 234.95 137.16) (xy 245.11 137.16)
+			(xy 215.9 97.79) (xy 215.9 118.11)
 		)
 		(stroke
@@
 	(wire
 		(pts
-			(xy 215.9 97.79) (xy 215.9 118.11)
+			(xy 115.57 63.5) (xy 115.57 73.66)
 		)
 		(stroke
@@
 	(wire
 		(pts
-			(xy 115.57 64.77) (xy 115.57 73.66)
-		)
-		(stroke
-			(width 0)
-			(type default)
-		)
-	)
-	(wire
-		(pts
 			(xy 41.91 86.36) (xy 59.69 86.36)
 		)
@@
 	(wire
 		(pts
-			(xy 115.57 46.99) (xy 115.57 57.15)
+			(xy 115.57 46.99) (xy 115.57 60.96)
 		)
 		(stroke
@@
 	)
 	(symbol
+		(lib_id "Connector_Audio:AudioJack2")
+		(at 120.65 63.5 0)
+		(mirror y)
+		(unit 1)
+		(exclude_from_sim no)
+		(in_bom yes)
+		(on_board yes)
+		(dnp no)
+		(property "Reference" "LS1"
+			(at 121.285 54.61 0)
+			(effects
+				(font
+					(size 1.27 1.27)
+				)
+			)
+		)
+		(property "Value" "Earphone"
+			(at 121.285 57.15 0)
+			(effects
+				(font
+					(size 1.27 1.27)
+				)
+			)
+		)
+		(property "Footprint" "SJ1_2503A:CONN_SJ1-2503A"
+			(at 120.65 63.5 0)
+			(effects
+				(font
+					(size 1.27 1.27)
+				)
+				(hide yes)
+			)
+		)
+		(property "Datasheet" "~"
+			(at 120.65 63.5 0)
+			(effects
+				(font
+					(size 1.27 1.27)
+				)
+				(hide yes)
+			)
+		)
+		(property "Description" "Audio Jack, 2 Poles (Mono / TS)"
+			(at 120.65 63.5 0)
+			(effects
+				(font
+					(size 1.27 1.27)
+				)
+				(hide yes)
+			)
+		)
+		(pin "T"
+		)
+		(pin "S"
+		)
+		(instances
+			(project ""
+				(path "/e63e39d7-6ac0-4ffd-8aa3-1841a4541b55"
+					(reference "LS1")
+					(unit 1)
+				)
+			)
+		)
+	)
+	(symbol
 		(lib_id "MCU_Module:Arduino_Nano_v3.x")
 		(at 72.39 99.06 180)
@@
 					(unit 1)
 				)
-			)
-		)
-	)
-	(symbol
-		(lib_id "Device:Earphone")
-		(at 115.57 62.23 0)
-		(unit 1)
-		(exclude_from_sim no)
-		(in_bom yes)
-		(on_board yes)
-		(dnp no)
-		(fields_autoplaced yes)
-		(property "Reference" "LS1"
-			(at 118.11 59.6899 0)
-			(effects
-				(font
-					(size 1.27 1.27)
-				)
-				(justify left)
-			)
-		)
-		(property "Value" "Earphone"
-			(at 118.11 62.2299 0)
-			(effects
-				(font
-					(size 1.27 1.27)
-				)
-				(justify left)
-			)
-		)
-		(property "Footprint" "SJ1_2503A:CONN_SJ1-2503A"
-			(at 115.57 59.69 90)
-			(effects
-				(font
-					(size 1.27 1.27)
-				)
-				(hide yes)
-			)
-		)
-		(property "Datasheet" "~"
-			(at 115.57 59.69 90)
-			(effects
-				(font
-					(size 1.27 1.27)
-				)
-				(hide yes)
-			)
-		)
-		(property "Description" "Earphone, polarized"
-			(at 115.57 62.23 0)
-			(effects
-				(font
-					(size 1.27 1.27)
-				)
-				(hide yes)
-			)
-		)
-		(pin "1"
-		)
-		(pin "2"
-		)
-		(instances
-			(project ""
-				(path "/e63e39d7-6ac0-4ffd-8aa3-1841a4541b55"
-					(reference "LS1")
-					(unit 1)
-				)
